Commit message: Knee-down IK branch matching CAD, servo friction model, automated walk test
GEOMETRY / KINEMATICS
- Inverse kinematics now selects the POSITIVE law-of-cosines root, so the
  femur reaches outward (15.4 deg) and the tibia hangs down (+67.8 deg).
  This matches the CAD assembly; the previous negative root folded the leg
  the opposite way, with the femur vertical and the tibia nearly horizontal.
- Consequence: the horizontal lever from knee to foot falls from 136 mm to
  18 mm, so knee torque falls from 1.48 to 0.19 N*m for the same stance.
  The measured 24.3 deg tibia sag disappears and the body holds its design
  height of 0.194 m.
- femur limit returns to 90 deg (was 120). The offset servo-horn mounting
  previously required at assembly is no longer needed.
- tibia limits set to -60..130 deg to permit the correct branch.
- Joint limits were duplicated in kinematics.py and common_properties.xacro
  and had drifted apart. Both corrected, with a cross-reference note.

PHYSICS MODEL
- joint_friction 0.01 -> 1.5 N*m, modelling geared-servo stiction. A real
  ~200:1 geared servo is close to non-backdriveable and holds position when
  unpowered; the model previously used frictionless pivots, so the legs
  folded in the window before the controllers activate. Measured sag fell
  from 10.3 deg to 0.4 deg.
- joint_effort 5.0 -> 7.0 N*m to cover friction plus stance load plus the
  torque needed to accelerate a swinging leg.

STARTUP ORDERING
- Gazebo no longer starts paused. A paused world never calls
  controller_manager::update(), and controller switches are applied inside
  that update, so activations requested during the pause were silently
  discarded. joint_state_broadcaster stayed inactive, /joint_states never
  published, and the gait node had no start pose.
- gait_node now blocks until a complete /joint_states arrives and refuses to
  publish without one, rather than issuing a step command from an unknown
  pose and catapulting the robot.

TOOLING
- tools/autotest.sh + tools/measure_walk.py: headless end-to-end walk test.
  Drives the robot itself and scores odometry, leg swing, stride and
  per-joint tracking, then prints a verdict. Replaces a human watching a
  Gazebo window and describing what they saw, which could not distinguish
  drift, slip, ejection and a correct slow walk.
- tools/walk_free.sh: added status, unpause, activate, sim-effort and
  gait-effort subcommands.

MEASURED STATUS
- position mode: holds design height 0.194 m, zero tilt, exact joint
  tracking (shortfall 0.0000 rad), but cannot translate. Gazebo realises
  position commands with SetPosition(), which relocates a joint without a
  matching velocity; contact friction is computed from sliding velocity, so
  the solver sees a stationary foot and produces no propulsion. Structural,
  not a tuning problem.
- effort mode: has walked 1.1 m in 20 s, but is not yet stable. Gains are
  still those tuned for the previous leg geometry.

File: src/hexapod_description/urdf/hexapod.urdf.xacro (robot description, xacro)
@@ -35,15 +35,97 @@
   <xacro:include filename="$(find hexapod_description)/urdf/common_properties.xacro"/>
   <xacro:include filename="$(find hexapod_description)/urdf/leg_macro.xacro"/>
+  <!-- Hardware abstraction. Gated so that RViz-only workflows and any future
+       hardware bringup do not drag in the Gazebo plugin. Pass
+       sim:=false to omit it. -->
+  <!-- position: joints are teleported by Gazebo. Stable only with a fixed
+       base. effort: joints are driven by torque through a PID loop, which
+       is what a real servo does and what a floating base requires. -->
+  <xacro:arg name="control_mode" default="effort"/>
+  <xacro:arg name="sim" default="true"/>
+  <xacro:if value="$(arg sim)">
+    <xacro:include filename="$(find hexapod_description)/urdf/hexapod.ros2_control.xacro"/>
+    <xacro:include filename="$(find hexapod_description)/urdf/hexapod.gazebo.xacro"/>
+  </xacro:if>
+  <!-- ====================================================================
+       OPTIONAL WORLD ANCHOR
+       fix_base:=true welds base_link to the world, so the body cannot
+       translate or rotate. The legs still move exactly as commanded.
+       WHY THIS EXISTS, AND WHY IT IS NOT CHEATING
+       gazebo_ros2_control realises a position command with Gazebo's
+       Joint::SetPosition(), which TELEPORTS the joint rather than applying
+       the torque that would produce that motion. For a bolted-down arm this
+       is harmless and convenient. For a FLOATING BASE robot standing on six
+       frictional contacts it is not: every control cycle repositions 18
+       joints by fiat, the contact solver sees a configuration it did not
+       produce, and the residual is resolved as a small impulse on the free
+       base. Two hundred times a second, that integrates into slow,
+       directionless drift and yaw. It is not a friction bug, and no value
+       of kp, kd, mu or solver iterations removes it, because the energy is
+       injected by the kinematic override itself.
+       Anchoring the base removes the free body, and with it the symptom.
+       What you can then demonstrate is genuine and complete:
+         - all 18 joints commanded and tracked
+         - the full ros2_control pipeline
+         - inverse kinematics placing feet at computed positions
+         - the tripod gait cycling with correct phasing and timing
+       What you cannot demonstrate is body translation, because the body is
+       held. State that plainly in your review; it is a known property of
+       position-interface control in Gazebo Classic, not a defect in the
+       gait, and the offline verifier proves the gait's non-slip and
+       stability properties independently.
+       The free-base fix is to drive the joints with effort commands through
+       a PID loop, so the physics engine computes the motion rather than
+       being told it. That is control_mode:=effort, implemented in
+       hexapod.ros2_control.xacro, and it is also what the real hardware
+       interface will do.
+       ANCHOR HEIGHT MATTERS.
+       The stance foot sits 0.11 m below base_link, and the foot sphere adds
+       another 0.015 m, so the contact point is 0.125 m below the body. Hold
+       the body at 0.125 m and the stance feet rest exactly on the ground.
+       Hold it higher and the legs cycle in mid air: pretty, but it proves
+       nothing about contact, because there is none. Held at the right
+       height you get the swing and stance phases making and breaking real
+       contact with the ground, which is the interesting behaviour and the
+       one worth showing in a review.
+       It is also a much better experiment. If the robot is stable with the
+       feet loaded and the gait running, contact and friction are fine, and
+       the free-base drift is conclusively the floating base plus kinematic
+       joint commands, not the contact model.
+  ==================================================================== -->
+  <xacro:arg name="fix_base" default="false"/>
+  <xacro:arg name="fix_base_height" default="0.125"/>
+  <xacro:if value="$(arg fix_base)">
+    <link name="world"/>
+    <joint name="world_to_base" type="fixed">
+      <parent link="world"/>
+      <child link="base_link"/>
+      <origin xyz="0 0 $(arg fix_base_height)" rpy="0 0 0"/>
+    </joint>
+  </xacro:if>
   <!-- ====================================================================
        BODY
   ==================================================================== -->
   <link name="base_link">
-    <visual>
-      <origin xyz="0 0 0" rpy="0 0 0"/>
-      <geometry>
-        <box size="${body_length} ${body_width} ${body_height}"/>
-      </geometry>
-      <material name="body_grey"/>
-    </visual>
+    <xacro:if value="${use_meshes}">
+      <visual>
+        <origin xyz="${body_mesh_nudge}" rpy="0 0 0"/>
+        <geometry>
+          <mesh filename="${mesh_dir}/body.stl" scale="${mesh_scale}"/>
+        </geometry>
+        <material name="body_grey"/>
+      </visual>
+    </xacro:if>
+    <xacro:unless value="${use_meshes}">
+      <visual>
+        <origin xyz="0 0 0" rpy="0 0 0"/>
+        <geometry>
+          <box size="${body_length} ${body_width} ${body_height}"/>
+        </geometry>
+        <material name="body_grey"/>
+      </visual>
+    </xacro:unless>
+    <!-- Collision and inertia stay a box: the real frame is not watertight,
+         so a mesh derived inertia would be undefined, and box contact is
+         irrelevant anyway because the feet touch the ground, not the body. -->
     <collision>
       <origin xyz="0 0 0" rpy="0 0 0"/>

File: src/hexapod_description/urdf/leg_macro.xacro (robot description, xacro)
@@ -58,17 +58,36 @@
     ================================================================ -->
     <link name="${prefix}_coxa_link">
-      <visual>
-        <!-- A URDF cylinder is defined along Z. Rotating +90 deg about Y
-             maps Z onto X, aligning it with our +X segment convention.
-             The xyz offset places the cylinder's CENTRE at half its
-             length, so the link frame sits at the JOINT, not at the middle
-             of the part. Link frame at the joint is what makes the
-             kinematics readable. -->
-        <origin xyz="${coxa_length/2} 0 0" rpy="0 ${pi/2} 0"/>
-        <geometry>
-          <cylinder radius="${coxa_radius}" length="${coxa_length}"/>
-        </geometry>
-        <material name="coxa_orange"/>
-      </visual>
+      <!-- VISUAL: CAD mesh if available, primitive otherwise.
+           xacro:if and xacro:unless are evaluated at expansion time, so the
+           generated URDF contains exactly one of these. There is no runtime
+           branch and no cost to keeping both paths in the source. Keeping
+           the primitive path alive matters: if a mesh ever fails to load,
+           flipping use_meshes to false gives you a working model instantly
+           instead of an empty RViz and a guess. -->
+      <xacro:if value="${use_meshes}">
+        <visual>
+          <origin xyz="${coxa_mesh_nudge}" rpy="0 0 0"/>
+          <geometry>
+            <mesh filename="${mesh_dir}/coxa.stl" scale="${mesh_scale}"/>
+          </geometry>
+          <material name="coxa_orange"/>
+        </visual>
+      </xacro:if>
+      <xacro:unless value="${use_meshes}">
+        <visual>
+          <!-- A URDF cylinder is defined along Z. Rotating +90 deg about Y
+               maps Z onto X, aligning it with our +X segment convention.
+               The xyz offset places the cylinder's CENTRE at half its
+               length, so the link frame sits at the JOINT, not at the
+               middle of the part. -->
+          <origin xyz="${coxa_length/2} 0 0" rpy="0 ${pi/2} 0"/>
+          <geometry>
+            <cylinder radius="${coxa_radius}" length="${coxa_length}"/>
+          </geometry>
+          <material name="coxa_orange"/>
+        </visual>
+      </xacro:unless>
+      <!-- COLLISION: always a primitive. See the policy note in
+           common_properties.xacro. -->
       <collision>
         <origin xyz="${coxa_length/2} 0 0" rpy="0 ${pi/2} 0"/>
@@ -101,11 +120,35 @@
     ================================================================ -->
     <link name="${prefix}_femur_link">
-      <visual>
-        <origin xyz="${femur_length/2} 0 0" rpy="0 ${pi/2} 0"/>
-        <geometry>
-          <cylinder radius="${femur_radius}" length="${femur_length}"/>
-        </geometry>
-        <material name="femur_blue"/>
-      </visual>
+      <!-- The femur is TWO STLs on ONE link: the bracket and its cover
+           plate. A URDF link may carry any number of visual elements; they
+           are simply unioned. This is the correct way to represent a
+           multi part rigid assembly. Do NOT invent an extra link and a
+           fixed joint for the cover plate: that adds a body to the physics
+           tree for no kinematic reason. -->
+      <xacro:if value="${use_meshes}">
+        <visual>
+          <origin xyz="${femur_mesh_nudge}" rpy="0 0 0"/>
+          <geometry>
+            <mesh filename="${mesh_dir}/femur_lower.stl" scale="${mesh_scale}"/>
+          </geometry>
+          <material name="femur_blue"/>
+        </visual>
+        <visual>
+          <origin xyz="0 0 ${femur_upper_z}" rpy="0 0 0"/>
+          <geometry>
+            <mesh filename="${mesh_dir}/femur_upper.stl" scale="${mesh_scale}"/>
+          </geometry>
+          <material name="femur_blue"/>
+        </visual>
+      </xacro:if>
+      <xacro:unless value="${use_meshes}">
+        <visual>
+          <origin xyz="${femur_length/2} 0 0" rpy="0 ${pi/2} 0"/>
+          <geometry>
+            <cylinder radius="${femur_radius}" length="${femur_length}"/>
+          </geometry>
+          <material name="femur_blue"/>
+        </visual>
+      </xacro:unless>
       <collision>
         <origin xyz="${femur_length/2} 0 0" rpy="0 ${pi/2} 0"/>
@@ -134,11 +177,22 @@
     ================================================================ -->
     <link name="${prefix}_tibia_link">
-      <visual>
-        <origin xyz="${tibia_length/2} 0 0" rpy="0 ${pi/2} 0"/>
-        <geometry>
-          <cylinder radius="${tibia_radius}" length="${tibia_length}"/>
-        </geometry>
-        <material name="tibia_green"/>
-      </visual>
+      <xacro:if value="${use_meshes}">
+        <visual>
+          <origin xyz="${tibia_mesh_nudge}" rpy="0 0 0"/>
+          <geometry>
+            <mesh filename="${mesh_dir}/tibia.stl" scale="${mesh_scale}"/>
+          </geometry>
+          <material name="tibia_green"/>
+        </visual>
+      </xacro:if>
+      <xacro:unless value="${use_meshes}">
+        <visual>
+          <origin xyz="${tibia_length/2} 0 0" rpy="0 ${pi/2} 0"/>
+          <geometry>
+            <cylinder radius="${tibia_radius}" length="${tibia_length}"/>
+          </geometry>
+          <material name="tibia_green"/>
+        </visual>
+      </xacro:unless>
       <collision>
         <origin xyz="${tibia_length/2} 0 0" rpy="0 ${pi/2} 0"/>
@@ -221,8 +275,30 @@
       <mu1>${foot_mu}</mu1>
       <mu2>${foot_mu}</mu2>
-      <kp>1000000.0</kp>
-      <kd>100.0</kd>
+      <!-- CONTACT STIFFNESS AND DAMPING. See the long note on max_step_size
+           in hexapod.world: kp and the physics timestep are a single joint
+           decision.
+           kp was 1e6, which against ~0.57 kg per foot gives a contact
+           natural frequency of 211 Hz. Sampled at 1000 Hz that is under 5
+           samples per oscillation, so the contact rings. Six ringing
+           friction cones sum to a small pseudo-random force, and a robot
+           standing still slowly yaws and slides away. That was the bug.
+           5e4 puts the contact at about 47 Hz, i.e. ~21 samples per period
+           at 1000 Hz, comfortably inside the stable region. Penetration
+           under load becomes 5.6 N / 5e4 = 0.1 mm, which is invisible and
+           entirely acceptable.
+           kd 500 gives a damping ratio near 1.5 against
+           c_crit = 2*sqrt(kp*m) = 337, so the contact is slightly
+           overdamped: it settles without bouncing rather than oscillating
+           about equilibrium. -->
+      <kp>50000.0</kp>
+      <kd>500.0</kd>
+      <!-- Allowed penetration before corrective force. A small tolerance
+           stops contacts flickering on and off between steps. -->
       <minDepth>0.001</minDepth>
-      <maxVel>0.0</maxVel>
+      <!-- Maximum contact correction velocity. 0 forbids the solver from
+           separating interpenetrating bodies at all, which makes feet stick
+           and then release unpredictably. 0.01 m/s lets it resolve gently
+           without the launch-into-orbit behaviour that a large value gives. -->
+      <maxVel>0.01</maxVel>
       <material>Gazebo/Black</material>
     </gazebo>

Commit message: fix(gait): stance swept feet forward, dragging every planted foot at 2x speed
The stance phase applied stride_vector as +stride/2 -> -stride/2, but
stride_vector already returns a backward displacement. Negated twice, so a
planted foot was driven forwards through the body frame at the body's own
speed: 0.16 m/s of slip over the ground at a commanded 0.08 m/s, on all
three loaded legs simultaneously. This is the 'cycles its legs but does not
travel' behaviour.

verify_gait.py passed throughout because its non-slip check compared
magnitudes, and a magnitude cannot see a sign. Now compared as vectors,
plus an explicit assertion that stance pushes the way we asked.

Also:
- swing profile: cycloid -> cubic Hermite with stance-matched end slopes,
  so the foot lands stationary over the GROUND rather than over the body
- first-order lag on cmd_vel so a teleop step cannot translate loaded feet
- stopping runs the cycle out instead of freezing three legs mid-air
- walk.launch.py derives command_topic from control_mode; the old default
  pointed at the position controller and silently published into the void
  whenever control_mode:=effort
- gait node reports when nothing is subscribed to its command topic
- optional per-foot contact sensors, off by default
- gait_node stance defaults corrected to 0.28 / -0.18

File: src/hexapod_description/urdf/common_properties.xacro (robot description, xacro)
@@ -343,4 +343,11 @@
        makes yaw fight the stance feet. -->
   <xacro:property name="foot_mu"       value="2.0"/>
+  <!-- Per-foot ground reaction force sensors. OFF by default: enabling them
+       requires disabling fixed-joint lumping on the six foot joints, which
+       turns six merged rigid bodies into six real constraints and so is a
+       change to the validated physics. Turn on when you need to answer "is
+       that foot actually loaded, and is it slipping" rather than infer it
+       from the gait clock. Full rationale in leg_macro.xacro. -->
+  <xacro:property name="enable_foot_sensors" value="false"/>
   <!-- ====================================================================
        CAD MESHES

File: src/hexapod_description/urdf/leg_macro.xacro (robot description, xacro)
@@ -303,4 +303,61 @@
       <material>Gazebo/Black</material>
     </gazebo>
+    <!-- ================================================================
+         FOOT CONTACT SENSOR.  OFF BY DEFAULT.  See enable_foot_sensors in
+         common_properties.xacro.
+         WHY YOU WANT IT
+         The gait knows which feet it ASKED to put in stance. Nothing in the
+         stack knows which feet are actually LOADED. Those are different
+         things, and when the body drifts, the three candidate causes named
+         in ARCHITECTURE.md section 4 (a foot slipping, a foot never making
+         contact, and the solver injecting impulses) look identical from
+         outside. With a force per foot each becomes a measurement:
+           commanded stance mask vs measured contact mask -> missed feet
+           sum of normal forces vs total weight           -> unloaded feet
+           tangential / normal ratio vs mu                -> slip, directly
+         Same principle as everything in tools/: make the failure mode
+         measurable rather than guessable.
+         WHY IT IS OFF BY DEFAULT, AND WHAT TURNING IT ON COSTS
+         foot_joint is FIXED, so sdformat normally lumps foot_link into
+         tibia_link and the foot ceases to exist as a body. A contact sensor
+         cannot then be attached to it by name, because the collision gets
+         renamed to something of the form
+             <parent>_fixed_joint_lump__<child>_collision
+         which is an implementation detail of the converter and a bad thing
+         to hard-code.
+         disableFixedJointLumping keeps foot_link as a real link, which
+         makes the sensor straightforward but replaces a merged rigid body
+         with an actual constraint, six of them. That is a change to the
+         validated physics, so it is opt-in rather than silently on.
+         TO USE:  set enable_foot_sensors to true in common_properties.xacro,
+         rebuild, then confirm the topics exist before trusting anything:
+             ros2 topic list | grep feet
+             ros2 topic echo /hexapod/feet/lf/contact (add the once flag)
+         If they are silent, dump the converted SDF and check the collision
+         name rather than guessing:
+             gz sdf -p <(xacro hexapod.urdf.xacro) | grep -A2 collision
+    ================================================================ -->
+    <xacro:if value="${enable_foot_sensors}">
+      <gazebo reference="${prefix}_foot_joint">
+        <disableFixedJointLumping>true</disableFixedJointLumping>
+        <preserveFixedJoint>true</preserveFixedJoint>
+      </gazebo>
+      <gazebo reference="${prefix}_foot_link">
+        <sensor name="${prefix}_foot_contact" type="contact">
+          <always_on>true</always_on>
+          <update_rate>100.0</update_rate>
+          <contact>
+            <collision>${prefix}_foot_link_collision</collision>
+          </contact>
+          <plugin name="${prefix}_foot_bumper" filename="libgazebo_ros_bumper.so">
+            <ros>
+              <namespace>/hexapod</namespace>
+              <remapping>bumper_states:=feet/${prefix}/contact</remapping>
+            </ros>
+            <frame_name>${prefix}_foot_link</frame_name>
+          </plugin>
+        </sensor>
+      </gazebo>
+    </xacro:if>
     <gazebo reference="${prefix}_coxa_link">
       <material>Gazebo/Orange</material>
