Commit message: feat(sim): sim_profile:=repo mirrors hexapod_ros physical assumptions
Adds a switch selecting which set of physical assumptions the model is
built with. Default is unchanged.

  physical  measured masses, closed-form inertias, derived joint limits,
            our tuned gains. What the report is about.
  repo      KevinOchs/hexapod_ros: 1e-5 kg links, identity inertia tensors,
            plus/minus pi limits, 6 N m / 0.524 rad/s, no joint dynamics,
            p=100 i=0 d=0.

repo mode is non-physical and stable because of it: gravity torque at 1e-5 kg
is negligible so a crude PID has thousands of times the authority it needs,
and a 1.0 kg m^2 tensor on such a link is far too reluctant to rotate for
anything to destabilise. It produces a robot that walks on screen and no
number that means anything about the real machine.

The controller YAML follows sim_profile automatically. Gains and masses are
one decision, not two.

Also adds docs/RUNBOOK.md, including the observation that the recorded
conclusion 'position + free base does not travel' was reached while the
stance swept the feet backwards, and is therefore void.

File: src/hexapod_description/urdf/common_properties.xacro (robot description, xacro)
@@ -392,4 +392,65 @@
   <xacro:property name="body_mesh_nudge"  value="0 0 0"/>
   <!-- ====================================================================
+       SIM PROFILE OVERRIDES
+       ====================================================================
+       sim_profile:=physical   (default)  our measured model
+       sim_profile:=repo                  KevinOchs/hexapod_ros assumptions
+       WHAT repo MODE DOES, AND WHAT IT COSTS
+       hexapod_ros gives every link a mass of 1e-5 kg and an identity
+       inertia tensor. Nothing about that is physical. It works, and it
+       works for a specific reason worth understanding: with negligible
+       mass the gravity torque on each link is negligible, so a crude PID
+       holds any pose effortlessly, and with an inertia tensor of 1.0
+       kg m^2 against a 1e-5 kg link the rotational inertia is enormous
+       relative to every force acting on it. The model is so heavily
+       damped by its own numbers that it cannot become unstable. It is a
+       kinematic animation wearing a physics engine as a coat.
+       That is the trade being made here deliberately: a robot that
+       visibly walks, in exchange for a simulation that can no longer tell
+       you anything true about torques, contact forces, servo sizing or
+       whether the real machine would stand up.
+       EVERYTHING IS RECOVERABLE. This block only overrides values. Launch
+       without sim_profile:=repo and the measured model is back, untouched.
+       The physical numbers below are still the ones in the report.
+       These overrides must stay AFTER the definitions above; xacro takes
+       the last assignment.
+  ==================================================================== -->
+  <xacro:arg name="sim_profile" default="physical"/>
+  <xacro:property name="sim_profile" value="$(arg sim_profile)"/>
+  <xacro:property name="repo_mode"   value="${sim_profile == 'repo'}"/>
+  <xacro:if value="${repo_mode}">
+    <!-- Masses. hexapod_ros uses 0.00001 kg for every link including the
+         body. Kept non-zero for the same reason their model does: a zero
+         mass link carrying a collision shape is a singular mass matrix. -->
+    <xacro:property name="body_mass"  value="0.00001"/>
+    <xacro:property name="coxa_mass"  value="0.00001"/>
+    <xacro:property name="femur_mass" value="0.00001"/>
+    <xacro:property name="tibia_mass" value="0.00001"/>
+    <!-- Joint limits. Theirs are plus/minus pi on every joint, which
+         discards the mechanical range we derived. The IK still respects
+         the real limits via kinematics.py, so this only removes the URDF
+         as a second line of defence. -->
+    <xacro:property name="coxa_lower"  value="${-pi}"/>
+    <xacro:property name="coxa_upper"  value="${ pi}"/>
+    <xacro:property name="femur_lower" value="${-pi}"/>
+    <xacro:property name="femur_upper" value="${ pi}"/>
+    <xacro:property name="tibia_lower" value="${-pi}"/>
+    <xacro:property name="tibia_upper" value="${ pi}"/>
+    <!-- Their AX-12 style numbers: 6 N m, 0.524 rad/s. The velocity limit
+         is 11x lower than ours and is doing real work in their model, by
+         capping how fast a joint can be driven at all. -->
+    <xacro:property name="joint_effort"   value="6.0"/>
+    <xacro:property name="joint_velocity" value="0.524"/>
+    <!-- Their URDF carries no <dynamics> tag at all. -->
+    <xacro:property name="joint_damping"  value="0.0"/>
+    <xacro:property name="joint_friction" value="0.0"/>
+  </xacro:if>
+  <!-- Mesh collision geometry, as hexapod_ros uses. Left OFF even in repo
+       mode: contact is evaluated pairwise across 25 links every physics
+       step, so swapping primitives for a 9,572 triangle mesh costs three
+       orders of magnitude and buys nothing, and their meshes are not
+       watertight either. Set true if you want the comparison. -->
+  <xacro:property name="repo_mesh_collision" value="false"/>
+  <!-- ====================================================================
        INERTIA MACROS
        Closed form inertia tensors for primitive solids, about the solid's
@@ -403,13 +464,29 @@
   ==================================================================== -->
   <!-- Solid cuboid, sides x, y, z, about its centre. -->
+  <!-- Identity tensor, repo mode only. hexapod_ros writes
+       ixx=iyy=izz=1.0 on every single link regardless of its size or mass.
+       Against a 1e-5 kg link that is roughly 100,000 times too large, which
+       is the actual reason their simulation never destabilises: every link
+       is far too reluctant to rotate for anything to go wrong. -->
   <xacro:macro name="inertial_box" params="mass x y z *origin">
-    <inertial>
-      <xacro:insert_block name="origin"/>
-      <mass value="${mass}"/>
-      <inertia
-        ixx="${(1.0/12.0) * mass * (y*y + z*z)}" ixy="0.0" ixz="0.0"
-        iyy="${(1.0/12.0) * mass * (x*x + z*z)}" iyz="0.0"
-        izz="${(1.0/12.0) * mass * (x*x + y*y)}"/>
-    </inertial>
+    <xacro:if value="${repo_mode}">
+      <inertial>
+        <xacro:insert_block name="origin"/>
+        <mass value="${mass}"/>
+        <inertia ixx="1.0" ixy="0.0" ixz="0.0"
+                 iyy="1.0" iyz="0.0"
+                 izz="1.0"/>
+      </inertial>
+    </xacro:if>
+    <xacro:unless value="${repo_mode}">
+      <inertial>
+        <xacro:insert_block name="origin"/>
+        <mass value="${mass}"/>
+        <inertia
+          ixx="${(1.0/12.0) * mass * (y*y + z*z)}" ixy="0.0" ixz="0.0"
+          iyy="${(1.0/12.0) * mass * (x*x + z*z)}" iyz="0.0"
+          izz="${(1.0/12.0) * mass * (x*x + y*y)}"/>
+      </inertial>
+    </xacro:unless>
   </xacro:macro>
   <!-- Solid cylinder whose axis of symmetry lies along X.
@@ -419,23 +496,45 @@
        right. -->
   <xacro:macro name="inertial_cylinder_x" params="mass radius length *origin">
-    <inertial>
-      <xacro:insert_block name="origin"/>
-      <mass value="${mass}"/>
-      <inertia
-        ixx="${0.5 * mass * radius * radius}" ixy="0.0" ixz="0.0"
-        iyy="${(1.0/12.0) * mass * (3.0*radius*radius + length*length)}" iyz="0.0"
-        izz="${(1.0/12.0) * mass * (3.0*radius*radius + length*length)}"/>
-    </inertial>
+    <xacro:if value="${repo_mode}">
+      <inertial>
+        <xacro:insert_block name="origin"/>
+        <mass value="${mass}"/>
+        <inertia ixx="1.0" ixy="0.0" ixz="0.0"
+                 iyy="1.0" iyz="0.0"
+                 izz="1.0"/>
+      </inertial>
+    </xacro:if>
+    <xacro:unless value="${repo_mode}">
+      <inertial>
+        <xacro:insert_block name="origin"/>
+        <mass value="${mass}"/>
+        <inertia
+          ixx="${0.5 * mass * radius * radius}" ixy="0.0" ixz="0.0"
+          iyy="${(1.0/12.0) * mass * (3.0*radius*radius + length*length)}" iyz="0.0"
+          izz="${(1.0/12.0) * mass * (3.0*radius*radius + length*length)}"/>
+      </inertial>
+    </xacro:unless>
   </xacro:macro>
   <!-- Solid sphere about its centre. Used for the foot contact pad. -->
   <xacro:macro name="inertial_sphere" params="mass radius *origin">
-    <inertial>
-      <xacro:insert_block name="origin"/>
-      <mass value="${mass}"/>
-      <inertia
-        ixx="${0.4 * mass * radius * radius}" ixy="0.0" ixz="0.0"
-        iyy="${0.4 * mass * radius * radius}" iyz="0.0"
-        izz="${0.4 * mass * radius * radius}"/>
-    </inertial>
+    <xacro:if value="${repo_mode}">
+      <inertial>
+        <xacro:insert_block name="origin"/>
+        <mass value="0.00001"/>
+        <inertia ixx="1.0" ixy="0.0" ixz="0.0"
+                 iyy="1.0" iyz="0.0"
+                 izz="1.0"/>
+      </inertial>
+    </xacro:if>
+    <xacro:unless value="${repo_mode}">
+      <inertial>
+        <xacro:insert_block name="origin"/>
+        <mass value="${mass}"/>
+        <inertia
+          ixx="${0.4 * mass * radius * radius}" ixy="0.0" ixz="0.0"
+          iyy="${0.4 * mass * radius * radius}" iyz="0.0"
+          izz="${0.4 * mass * radius * radius}"/>
+      </inertial>
+    </xacro:unless>
   </xacro:macro>
   <!-- ====================================================================

File: src/hexapod_description/urdf/hexapod.ros2_control.xacro (robot description, xacro)
@@ -168,7 +168,18 @@
        install space, which $(find ...) provides.
   ==================================================================== -->
+  <!-- The controller YAML follows sim_profile, because the gains are only
+       meaningful against a particular set of masses. repo mode's p=100 is
+       tuned against 1e-5 kg links; applying it to the measured model gives
+       legs that cannot hold the robot up. Applying our gains to the repo
+       model gives an absurdly stiff joint. They are not interchangeable and
+       must not be selected independently. -->
   <gazebo>
     <plugin filename="libgazebo_ros2_control.so" name="gazebo_ros2_control">
-      <parameters>$(find hexapod_control)/config/controllers.yaml</parameters>
+      <xacro:if value="${repo_mode}">
+        <parameters>$(find hexapod_control)/config/controllers_repo.yaml</parameters>
+      </xacro:if>
+      <xacro:unless value="${repo_mode}">
+        <parameters>$(find hexapod_control)/config/controllers.yaml</parameters>
+      </xacro:unless>
       <robot_param>robot_description</robot_param>
       <robot_param_node>robot_state_publisher</robot_param_node>

Commit message: feat(demo): kinematic demonstration mode, body pose driven by the gait
DELIVERABLE FOR THE REVIEW. One command, robot walks, cannot be thrown.

Every Gazebo failure this project has had is one failure: a floating base on
six frictional contacts. Measured across three configurations:

  position + measured model    legs swing 10 deg, body travels 0.4 mm / 20 s
  effort   + hexapod_ros model walks at 99 percent tracking, climbs 5 cm,
                               tilts 12 deg
  effort   + measured model    body pinned at the origin, unresolved

What is demonstrably NOT at fault: the gait (498 offline assertions including
a signed non-slip test), the IK (round trip 3.5e-16 m), the URDF (mounts and
axes match kinematics.py exactly), and the controller (config B tracked
commanded angles to four decimals).

So the contact integration is the only unsolved part, and it is not on the
critical path for showing the gait works.

body_driver.py integrates the body pose from /cmd_vel using the SAME filter,
deadband and stance radius as GaitGenerator, imported rather than copied so
they cannot drift. sim_profile:=demo keeps every measured mass and inertia and
disables gravity only, so the solver does not fight the imposed pose.

This is not invented motion. The gait is provably non-slip: stance feet have
exactly zero velocity over the ground at every sampled phase. A planted foot
plus an advancing body therefore implies a body displacement, exactly, by
geometry. This integrates that displacement instead of having Gazebo
rediscover it through friction cones.

Present it as kinematic simulation. Do not quote torque, contact force, slip
or stability margin from it; those belong to sim_profile:=physical and are
reported separately as real findings.

File: src/hexapod_description/urdf/common_properties.xacro (robot description, xacro)
@@ -419,4 +419,23 @@
   <xacro:property name="sim_profile" value="$(arg sim_profile)"/>
   <xacro:property name="repo_mode"   value="${sim_profile == 'repo'}"/>
+  <!-- ====================================================================
+       sim_profile:=demo   KINEMATIC DEMONSTRATION MODE
+       ====================================================================
+       Masses, inertias and joint limits are the MEASURED ones, unchanged.
+       The only difference is that gravity is disabled per link.
+       WHY. In demo mode hexapod_gait/body_driver.py sets the body pose
+       directly from the gait, because the contact solver is the one part of
+       this stack nobody has made behave with a floating base. If gravity
+       stays on, every imposed pose is a teleport that the solver then tries
+       to correct, and the robot jitters or is thrown.
+       The legs still run the real gait and the real IK. Only the step where
+       Gazebo rediscovers the body displacement by integrating friction cones
+       is skipped, and that displacement is already guaranteed by the gait's
+       non-slip property, which verify_gait.py asserts at every sampled phase.
+       PRESENT THIS AS KINEMATIC SIMULATION. Do not quote a torque, a contact
+       force, a slip figure or a stability margin from it. Those come from
+       sim_profile:=physical, and the results there are reported separately.
+  ==================================================================== -->
+  <xacro:property name="demo_mode" value="${sim_profile == 'demo'}"/>
   <xacro:if value="${repo_mode}">
     <!-- Masses. hexapod_ros uses 0.00001 kg for every link including the

File: src/hexapod_description/urdf/hexapod.urdf.xacro (robot description, xacro)
@@ -140,4 +140,5 @@
   </link>
   <gazebo reference="base_link">
+    <xacro:if value="${demo_mode}"><gravity>0</gravity></xacro:if>
     <material>Gazebo/DarkGrey</material>
   </gazebo>

File: src/hexapod_description/urdf/leg_macro.xacro (robot description, xacro)
@@ -273,4 +273,5 @@
     ================================================================ -->
     <gazebo reference="${prefix}_foot_link">
+      <xacro:if value="${demo_mode}"><gravity>0</gravity></xacro:if>
       <mu1>${foot_mu}</mu1>
       <mu2>${foot_mu}</mu2>
@@ -361,10 +362,13 @@
     </xacro:if>
     <gazebo reference="${prefix}_coxa_link">
+      <xacro:if value="${demo_mode}"><gravity>0</gravity></xacro:if>
       <material>Gazebo/Orange</material>
     </gazebo>
     <gazebo reference="${prefix}_femur_link">
+      <xacro:if value="${demo_mode}"><gravity>0</gravity></xacro:if>
       <material>Gazebo/Blue</material>
     </gazebo>
     <gazebo reference="${prefix}_tibia_link">
+      <xacro:if value="${demo_mode}"><gravity>0</gravity></xacro:if>
       <material>Gazebo/Green</material>
     </gazebo>
