Commit message: Knee-down IK branch matching CAD, servo friction model, automated walk test
GEOMETRY / KINEMATICS
- Inverse kinematics now selects the POSITIVE law-of-cosines root, so the
  femur reaches outward (15.4 deg) and the tibia hangs down (+67.8 deg).
  This matches the CAD assembly; the previous negative root folded the leg
  the opposite way, with the femur vertical and the tibia nearly horizontal.
- Consequence: the horizontal lever from knee to foot falls from 136 mm to
  18 mm, so knee torque falls from 1.48 to 0.19 N*m for the same stance.
  The measured 24.3 deg tibia sag disappears and the body holds its design
  height of 0.194 m.
- femur limit returns to 90 deg (was 120). The offset servo-horn mounting
  previously required at assembly is no longer needed.
- tibia limits set to -60..130 deg to permit the correct branch.
- Joint limits were duplicated in kinematics.py and common_properties.xacro
  and had drifted apart. Both corrected, with a cross-reference note.

PHYSICS MODEL
- joint_friction 0.01 -> 1.5 N*m, modelling geared-servo stiction. A real
  ~200:1 geared servo is close to non-backdriveable and holds position when
  unpowered; the model previously used frictionless pivots, so the legs
  folded in the window before the controllers activate. Measured sag fell
  from 10.3 deg to 0.4 deg.
- joint_effort 5.0 -> 7.0 N*m to cover friction plus stance load plus the
  torque needed to accelerate a swinging leg.

STARTUP ORDERING
- Gazebo no longer starts paused. A paused world never calls
  controller_manager::update(), and controller switches are applied inside
  that update, so activations requested during the pause were silently
  discarded. joint_state_broadcaster stayed inactive, /joint_states never
  published, and the gait node had no start pose.
- gait_node now blocks until a complete /joint_states arrives and refuses to
  publish without one, rather than issuing a step command from an unknown
  pose and catapulting the robot.

TOOLING
- tools/autotest.sh + tools/measure_walk.py: headless end-to-end walk test.
  Drives the robot itself and scores odometry, leg swing, stride and
  per-joint tracking, then prints a verdict. Replaces a human watching a
  Gazebo window and describing what they saw, which could not distinguish
  drift, slip, ejection and a correct slow walk.
- tools/walk_free.sh: added status, unpause, activate, sim-effort and
  gait-effort subcommands.

MEASURED STATUS
- position mode: holds design height 0.194 m, zero tilt, exact joint
  tracking (shortfall 0.0000 rad), but cannot translate. Gazebo realises
  position commands with SetPosition(), which relocates a joint without a
  matching velocity; contact friction is computed from sliding velocity, so
  the solver sees a stationary foot and produces no propulsion. Structural,
  not a tuning problem.
- effort mode: has walked 1.1 m in 20 s, but is not yet stable. Gains are
  still those tuned for the previous leg geometry.

File: src/hexapod_description/urdf/hexapod.urdf.xacro (robot description, xacro)
@@ -109,5 +109,5 @@
     <xacro:if value="${use_meshes}">
       <visual>
-        <origin xyz="${body_mesh_nudge}" rpy="0 0 0"/>
+        <origin xyz="${body_mesh_nudge}" rpy="${body_mesh_rpy}"/>
         <geometry>
           <mesh filename="${mesh_dir}/body.stl" scale="${mesh_scale}"/>

File: src/hexapod_description/urdf/leg_macro.xacro (robot description, xacro)
@@ -67,6 +67,14 @@
       <xacro:if value="${use_meshes}">
         <visual>
-          <origin xyz="${coxa_mesh_nudge}" rpy="0 0 0"/>
-          <geometry>
+          <origin xyz="${coxa_mesh_nudge}" rpy="${coxa_mesh_rpy}"/>
+          <geometry>
+            <!-- NOT swapped. coxa.stl is the forked clevis at the LEFT end of
+                 the assembled CAD leg, the part that bolts to the body, so it
+                 belongs on the coxa link. An earlier revision exchanged this
+                 with the tibia visual on a misreading of the assembly photo;
+                 that exchange has been removed and the splitter's own naming
+                 is trusted again. split_assembly.py sorts the three
+                 components along +X with the body end lowest, so the file
+                 called coxa really is the proximal part. -->
             <mesh filename="${mesh_dir}/coxa.stl" scale="${mesh_scale}"/>
           </geometry>
@@ -120,25 +128,32 @@
     ================================================================ -->
     <link name="${prefix}_femur_link">
-      <!-- The femur is TWO STLs on ONE link: the bracket and its cover
-           plate. A URDF link may carry any number of visual elements; they
-           are simply unioned. This is the correct way to represent a
-           multi part rigid assembly. Do NOT invent an extra link and a
-           fixed joint for the cover plate: that adds a body to the physics
-           tree for no kinematic reason. -->
+      <!-- REVISION 2: the femur is a SINGLE part, 120 x 25 x 33 mm.
+           Revision 1 was a bracket plus a separate 5 mm cover plate, carried
+           as two <visual> elements on this one link with a stacking offset.
+           A URDF link may hold any number of visuals and they are simply
+           unioned, which was the right way to model that assembly. The new
+           CAD makes it one piece, so one visual. -->
       <xacro:if value="${use_meshes}">
         <visual>
-          <origin xyz="${femur_mesh_nudge}" rpy="0 0 0"/>
-          <geometry>
-            <mesh filename="${mesh_dir}/femur_lower.stl" scale="${mesh_scale}"/>
+          <origin xyz="${femur_mesh_nudge}" rpy="${femur_mesh_rpy}"/>
+          <geometry>
+            <mesh filename="${mesh_dir}/femur.stl" scale="${mesh_scale}"/>
           </geometry>
           <material name="femur_blue"/>
         </visual>
-        <visual>
-          <origin xyz="0 0 ${femur_upper_z}" rpy="0 0 0"/>
-          <geometry>
-            <mesh filename="${mesh_dir}/femur_upper.stl" scale="${mesh_scale}"/>
-          </geometry>
-          <material name="femur_blue"/>
-        </visual>
+        <!-- The repeated joint bracket. Same printed part as the coxa, used
+             again here. Rigidly bolted, so it is an extra visual on this
+             link rather than a link of its own: it has no degree of freedom
+             and giving it a fixed joint would add a body to the physics tree
+             for nothing. Its 21 g is already inside femur_mass. -->
+        <xacro:if value="${show_joint_brackets}">
+          <visual>
+            <origin xyz="${femur_bracket_xyz}" rpy="${femur_bracket_rpy}"/>
+            <geometry>
+              <mesh filename="${mesh_dir}/${bracket_mesh}" scale="${mesh_scale}"/>
+            </geometry>
+            <material name="coxa_orange"/>
+          </visual>
+        </xacro:if>
       </xacro:if>
       <xacro:unless value="${use_meshes}">
@@ -179,10 +194,24 @@
       <xacro:if value="${use_meshes}">
         <visual>
-          <origin xyz="${tibia_mesh_nudge}" rpy="0 0 0"/>
-          <geometry>
+          <origin xyz="${tibia_mesh_nudge}" rpy="${tibia_mesh_rpy}"/>
+          <geometry>
+            <!-- NOT swapped. tibia.stl is the trussed member at the RIGHT
+                 end of the assembled CAD leg, the one that carries the foot,
+                 so it belongs on the tibia link. See the matching note on
+                 the coxa link. -->
             <mesh filename="${mesh_dir}/tibia.stl" scale="${mesh_scale}"/>
           </geometry>
           <material name="tibia_green"/>
         </visual>
+        <!-- Third instance of the same bracket. Its 21 g is in tibia_mass. -->
+        <xacro:if value="${show_joint_brackets}">
+          <visual>
+            <origin xyz="${tibia_bracket_xyz}" rpy="${tibia_bracket_rpy}"/>
+            <geometry>
+              <mesh filename="${mesh_dir}/${bracket_mesh}" scale="${mesh_scale}"/>
+            </geometry>
+            <material name="coxa_orange"/>
+          </visual>
+        </xacro:if>
       </xacro:if>
       <xacro:unless value="${use_meshes}">
